Commit message: Road segmentation and autonomy demo

File: isaac_ros-dev/src/agv_bot_description/src/description/agv_bot_description.urdf (robot description, URDF)
Before this commit: robot agv_car, 3 links, 2 joints
Links:
- removed link lidar
- added link velodyne; visual cylinder length=.0762 radius=.0762
Joints:
- joint velodyne_joint: child lidar -> velodyne
